Commit message: Fixed Models in wrong folder

File: my_robot/urdf/my_robot.xacro (robot description, xacro)
@@ -56,4 +56,32 @@
     </visual>
   </link>
+  <link name='top_siren'>
+    <inertial>
+      <mass value="0.3"/>
+      <inertia
+          ixx="0.1" ixy="0" ixz="0"
+          iyy="0.1" iyz="0"
+          izz="0.1"
+      />
+    </inertial>
+    <visual name='top_siren_visual'>
+      <origin xyz="0 0 0" rpy="0 0 0"/>
+      <geometry>
+        <cylinder radius="0.05" length="0.02"/>
+      </geometry>
+    </visual>
+    <collision name='top_siren_visual'>
+      <origin xyz="0 0 0" rpy="0 0 0"/>
+      <geometry>
+        <cylinder radius="0.05" length="0.02"/>
+      </geometry>
+    </collision>
+  </link>
+  <joint type="fixed" name="top_siren_joint">
+    <origin xyz="-0.15 0 0.1" rpy="0 0 0"/>
+    <child link="top_siren"/>
+    <parent link="chassis"/>
+    <axis xyz="0 0 1" rpy="0 0 0"/>
+  </joint>
   <link name='left_wheel'>
     <inertial>
@@ -189,3 +217,9 @@
     <material>Gazebo/Red</material>
   </gazebo>
+  <gazebo reference="hokuyo">
+    <material>Gazebo/Gray</material>
+  </gazebo>
+  <gazebo reference="top_siren">
+    <material>Gazebo/Red</material>
+  </gazebo>
 </robot>
